File: pcb.NOT-READY.rounded/cheating-calc.kicad_pcb (KiCad board)
At the start: 2 copper layers, 72 x 22 mm, 16 parts, among them J1 Conn_01x04, J2 Conn_01x04, Q1 MMBF170, Q2 MMBF170, U1 ESP32-C3-MINI-1-N4, U2 AP7215-33YG-13

Commit message: update routing
Parts:
- C1, C2: value CL05A105KP5NNNC -> CL21B105KBFNNNE; footprint easyeda2kicad:C0402 -> easyeda2kicad:C0805
- moved C2 3.72 mm to (95.2, 65.0), turned to 90 degrees
- moved C1 3.63 mm to (88.2, 65.0), turned to -90 degrees
- moved U2 3.54 mm to (91.8, 64.3)
Routing:
- net +5V: track 85.5 -> 87.6 mm
- net GND: track 104.1 -> 105.5 mm
- net +3.3V: track 30.9 -> 31.6 mm
