File: InitialProgrammer/InitialProgrammer.kicad_pcb (KiCad board)
At the start: 2 copper layers, 24 x 20 mm, 7 parts, among them CN1 YZ29115060P-02, CN2 YZ29115060P-02, CN3 YZ29115060P-02, CN4 YZ29115060P-02, CN5 YZ29115060P-02, CN6 YZ29115060P-02

Commit message: update
Parts:
- moved CN1 16.6 mm to (152.0, 88.1)
- moved CN2 16.6 mm to (149.0, 88.1)
- moved CN3 16.6 mm to (146.0, 88.1)
- moved CN4 16.6 mm to (143.0, 88.1)
- moved CN5 16.6 mm to (140.0, 88.1)
- moved CN6 16.6 mm to (137.0, 88.1)
- moved H1 16.6 mm to (144.7, 99.8)
Other:
- board text added: "Converts https://www.tindie.com/products/snakeye/usb-programmer-for-esp8266esp32/ to pad format used by board."

Commit message: update
Other:
- board text added: "Converts ESP01 to pad format used by board."
- board text removed: "Converts https://www.tindie.com/products/snakeye/usb-programmer-for-esp8266esp32/ to pad format used by board."
Changed lines of the file:
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@@
 		(model "${EASYEDA2KICAD}/easyeda2kicad.3dshapes/TESTPOINT-SMD_BD2.0-D0.7.wrl"
 			(offset
-				(xyz 0 -0 2)
+				(xyz 0 -0 -2)
 			)
 			(scale
@@
 		(model "${EASYEDA2KICAD}/easyeda2kicad.3dshapes/TESTPOINT-SMD_BD2.0-D0.7.wrl"
 			(offset
-				(xyz 0 -0 2)
+				(xyz 0 -0 -2)
 			)
 			(scale
@@
 		(model "${EASYEDA2KICAD}/easyeda2kicad.3dshapes/TESTPOINT-SMD_BD2.0-D0.7.wrl"
 			(offset
-				(xyz 0 -0 2)
+				(xyz 0 -0 -2)
 			)
 			(scale
@@
 		(model "${EASYEDA2KICAD}/easyeda2kicad.3dshapes/TESTPOINT-SMD_BD2.0-D0.7.wrl"
 			(offset
-				(xyz 0 -0 2)
+				(xyz 0 -0 -2)
 			)
 			(scale
@@
 		(model "${EASYEDA2KICAD}/easyeda2kicad.3dshapes/TESTPOINT-SMD_BD2.0-D0.7.wrl"
 			(offset
-				(xyz 0 -0 2)
+				(xyz 0 -0 -2)
 			)
 			(scale
@@
 		(model "${EASYEDA2KICAD}/easyeda2kicad.3dshapes/TESTPOINT-SMD_BD2.0-D0.7.wrl"
 			(offset
-				(xyz 0 -0 2)
+				(xyz 0 -0 -2)
 			)
 			(scale
@@
 			)
 		)
+	)
+	(gr_circle
+		(center 154.2 88.099999)
+		(end 154.200001 88.099999)
+		(stroke
+			(width 1)
+			(type default)
+		)
+		(fill none)
+		(layer "B.SilkS")
+	)
+	(gr_circle
+		(center 138.6 101.1)
+		(end 138.600001 101.1)
+		(stroke
+			(width 1)
+			(type default)
+		)
+		(fill none)
+		(layer "B.SilkS")
+	)
+	(gr_circle
+		(center 154.2 88.099999)
+		(end 154.2 88.099999)
+		(stroke
+			(width 1)
+			(type default)
+		)
+		(fill none)
+		(layer "F.SilkS")
+	)
+	(gr_circle
+		(center 138.6 101.1)
+		(end 138.6 101.1)
+		(stroke
+			(width 1)
+			(type default)
+		)
+		(fill none)
+		(layer "F.SilkS")
 	)
 	(gr_rect
@@
 		)
 	)
-	(gr_text "Converts https://www.tindie.com/products/snakeye/usb-programmer-for-esp8266esp32/ to pad format used by board."
-		(at 99.5 110.1 0)
+	(gr_text "Converts ESP01 to pad format used by board."
+		(at 126.9 107.6 0)
 		(layer "Cmts.User")
 		(effects
