File: InitialProgrammer/InitialProgrammer.kicad_sch (KiCad schematic)
At the start: 7 parts, among them CN1 YZ29115060P-02, CN2 YZ29115060P-02, CN3 YZ29115060P-02, CN4 YZ29115060P-02, CN5 YZ29115060P-02, CN6 YZ29115060P-02

Commit message: update
Other:
- note added: "Converts https://www.tindie.com/products/snakeye/usb-programmer-for-esp8266esp32/ to pad format used by board"
- moved on the sheet: CN1, CN2, CN3, CN4, CN5, CN6, H1

Commit message: update
Other:
- note added: "Converts ESP01 to pad format used by board"
- note removed: "Converts https://www.tindie.com/products/snakeye/usb-programmer-for-esp8266esp32/ to pad format used by board"
Changed lines of the file:
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@@
 		)
 	)
-	(text "Converts https://www.tindie.com/products/snakeye/usb-programmer-for-esp8266esp32/ to pad format used by board"
+	(text "Converts ESP01 to pad format used by board"
 		(exclude_from_sim no)
-		(at 119.38 84.328 0)
+		(at 118.11 88.138 0)
 		(effects
 			(font
