File: pcb.alt.rounded/cheating-calc.kicad_sch (KiCad schematic)
At the start: 8 parts, among them J1 Conn_01x04, Q1 MMBF170, Q2 MMBF170, U1 XIAO-ESP32-S3-SMD

Commit message: update and add tht version
Parts:
- U1: symbol Seeed_Studio_XIAO_Series-20240814:XIAO-ESP32-C6-SMD -> Seeed_Studio_XIAO_Series:XIAO-ESP32-C6-SMD
Changed lines of the file:
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@@
 (kicad_sch
-	(version 20231120)
+	(version 20250114)
 	(generator "eeschema")
-	(generator_version "8.0")
+	(generator_version "9.0")
 	(paper "A4")
 	(junction
@@
 	)
 	(symbol
-		(lib_id "Seeed_Studio_XIAO_Series-20240814:XIAO-ESP32-C6-SMD")
+		(lib_id "Seeed_Studio_XIAO_Series:XIAO-ESP32-C6-SMD")
 		(at 179.07 88.9 0)
 		(unit 1)
@@
 		)
 	)
+	(embedded_fonts no)
 )
